Commit message: wip kuka grasp

File: python/examples/kuka_grasp/kuka_iiwa_gripper.urdf (robot description, URDF)
Before this commit: robot kuka_lbr_iiwa_14_r820, 12 links, 11 joints
Links:
- link base_link: geometry collision box size=0.257471 0.242590 0.157500; visual mesh filename=C:/dev/threepp/build/_deps/threepp_data-src/urdf/lbr_iiwa_1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
- link link_1: geometry collision box size=0.171682 0.202325 0.297430; visual mesh filename=C:/dev/threepp/build/_deps/threepp_data-src/urdf/lbr_iiwa_1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
- link link_2: geometry collision box size=0.171320 0.199618 0.289575; visual mesh filename=C:/dev/threepp/build/_deps/threepp_data-src/urdf/lbr_iiwa_1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
- link link_3: geometry collision box size=0.136049 0.182662 0.293272; visual mesh filename=C:/dev/threepp/build/_deps/threepp_data-src/urdf/lbr_iiwa_1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
- link link_4: geometry collision box size=0.136926 0.183015 0.252173; visual mesh filename=C:/dev/threepp/build/_deps/threepp_data-src/urdf/lbr_iiwa_1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
- link link_5: geometry collision box size=0.136273 0.167034 0.277175; visual mesh filename=C:/dev/threepp/build/_deps/threepp_data-src/urdf/lbr_iiwa_1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
- link link_6: geometry collision box size=0.132602 0.137681 0.167384; visual mesh filename=C:/dev/threepp/build/_deps/threepp_data-src/urdf/lbr_iiwa_1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
- link link_7: geometry collision box size=0.103694 0.103857 0.054917; visual mesh filename=C:/dev/threepp/build/_deps/threepp_data-src/urdf/lbr_iiwa_1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

Commit message: kuka_grasp: update scenario

File: python/examples/kuka_grasp/kuka_iiwa_gripper.urdf (robot description, URDF)
Before this commit: robot kuka_lbr_iiwa_14_r820, 12 links, 11 joints
Links:
- link base_link: geometry collision box size=0.257471 0.242590 0.157500; visual mesh filename=C:/dev/threepp/cmake-build-relwithdebinfo/_deps/threepp_dat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
- link link_1: geometry collision box size=0.171682 0.202325 0.297430; visual mesh filename=C:/dev/threepp/cmake-build-relwithdebinfo/_deps/threepp_dat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
- link link_2: geometry collision box size=0.171320 0.199618 0.289575; visual mesh filename=C:/dev/threepp/cmake-build-relwithdebinfo/_deps/threepp_dat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
- link link_3: geometry collision box size=0.136049 0.182662 0.293272; visual mesh filename=C:/dev/threepp/cmake-build-relwithdebinfo/_deps/threepp_dat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
- link link_4: geometry collision box size=0.136926 0.183015 0.252173; visual mesh filename=C:/dev/threepp/cmake-build-relwithdebinfo/_deps/threepp_dat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
- link link_5: geometry collision box size=0.136273 0.167034 0.277175; visual mesh filename=C:/dev/threepp/cmake-build-relwithdebinfo/_deps/threepp_dat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
- link link_6: geometry collision box size=0.132602 0.137681 0.167384; visual mesh filename=C:/dev/threepp/cmake-build-relwithdebinfo/_deps/threepp_dat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
- link link_7: geometry collision box size=0.103694 0.103857 0.054917; visual mesh filename=C:/dev/threepp/cmake-build-relwithdebinfo/_deps/threepp_dat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
